File: HW V1/RW612Implant/RW612Implant.kicad_sch (KiCad schematic)
At the start: 1 part, among them IC1 RW612ET

Commit message: clocked up on a saturday
Parts:
- added R1: 100R, Resistor_SMD:R_0201_0603Metric, symbol Device:R
- added Y1: 616L3I040M00000R, Library:616L3I008M00000R, symbol New_Library:616L3I040M00000R
Connections:
- net GND: now also R1.2, Y1.2 (Ground)
- net +3V3: now reaches IC1.A10 (VBAT_1)
- net +3V3: now also IC1.A4 (VIO_5), IC1.B10 (VBAT_2)
- net +1V8: now reaches IC1.B12 (AVDD18_1)
- net +1V8: now also IC1.D1 (VIO_4), IC1.F14 (AVDD18_2), IC1.F15 (AVDD18_3), IC1.J15 (AVDD18_4), IC1.K1 (VIO_1), IC1.K15 (AVDD18_5), IC1.L15 (AVDD18_6), IC1.M15 (AVDD18_7), IC1.N15 (AVDD18_8), IC1.P1 (AVDD18_9), IC1.R1 (AVDD18_10), IC1.R10 (AVDD18_12), IC1.R11 (AVDD18_13), IC1.R12 (AVDD18_14), IC1.R2 (AVDD18_11), Y1.1 (Enable), Y1.4 (Supply_Voltage)
- net at IC1.G15 (XTAL_OUT): now also R1.1
- net at IC1.H15 (XTAL_IN): now also Y1.3 (Output)

Commit message: we do a little routing
Connections:
- net +3V3: now also IC1.A5 (VIO_3), IC1.B15 (VIO_6)
- net LED_G: now reaches IC1.C5 (GPIO[27])
- net LED_R: now reaches IC1.F6 (GPIO[26])
- net LED_B: now reaches IC1.F8 (GPIO[4])
Other:
- sheet Peripherals ports: added LED_B, LED_G, LED_R; removed none

Commit message: everything except temp and qi?
Parts:
- added C10, C11, C12, C13, C14, C16, C17, C25, C27, C28, C29, C30, C8: 0.1u, Capacitor_SMD:C_0201_0603Metric, symbol Device:C
- added C15: 100p, Capacitor_SMD:C_0201_0603Metric, symbol Device:C
- added C18, C26: 470p, Capacitor_SMD:C_0201_0603Metric, symbol Device:C
- added C19, C20: 6TPS150MUD, Capacitor_Tantalum_SMD:CP_EIA-3528-21_Kemet-B, symbol Device:C_Polarized
- added C21, C22, C24, C31, C32: 22u X5R 6.3V, Capacitor_SMD:C_0402_1005Metric, symbol Device:C
- added J1: Conn_ARM_SWD_TagConnect_TC2030-NL, Connector:Tag-Connect_TC2030-IDC-NL_2x03_P1.27mm_Vertical, symbol Connector:Conn_ARM_SWD_TagConnect_TC2030-NL
- added L4, L5: LQM21PN1R0NGRD, Inductor_SMD:L_0805_2012Metric, symbol Device:L
- added R5: 50R, Resistor_SMD:R_0201_0603Metric, symbol Device:R
- added R6: 51k, Resistor_SMD:R_0201_0603Metric, symbol Device:R
Connections:
- net +1V8: now also IC1.C11 (BUCK18_SENSE), IC1.J13 (EXT_FREQ/WCI-2_SOUT), IC1.K13 (EXT_PRI), IC1.L13 (EXT_GNT), IC1.M12 (EXT_REQ), IC1.R6 (VIO_RF), C10.1, C11.1, C12.1, C13.1, C22.1, C30.1, C31.1, C8.1, L5.1
- net +3V3: now also IC1.B8 (AVDD33_USB), IC1.F1 (VIO_2), IC1.R15 (VPA_2), IC1.R8 (VPA_1), C14.1, C15.1, C16.1, C19.1, C20.1, C21.1, C27.1, C28.1, C29.1, J1.1 (VCC), R6.2
- net GND: now also IC1.P6 (RF_CNTL2), C10.2, C11.2, C12.2, C13.2, C14.2, C15.2, C16.2, C17.2, C18.2, C19.2, C20.2, C21.2, C22.2, C24.2, C25.2, C26.2, C27.2, C28.2, C29.2, C30.2, C31.2, C32.2, C8.2, J1.5 (GND), R5.2
- net at IC1.A11 (BUCK18_VOUT): now also L5.2
- net I2C_SCL: now reaches IC1.A14 (GPIO[56])
- net at IC1.A9 (BUCK11_VOUT): now also L4.2
- net I2C_SDA: now reaches IC1.B13 (GPIO[57])
- net +1V0: now reaches IC1.B9 (BUCK11_SENSE)
- net +1V0: now also IC1.D15 (VCORE_2), IC1.D4 (VCORE_1), IC1.H1 (VCORE_3), IC1.K10 (VCORE_4), C17.1, C18.1, C24.1, C25.1, C26.1, C32.1, L4.1
- net ~{RESET}: now reaches IC1.E9 (PDN)
- net ~{RESET}: now also J1.3 (~{RESET}), R6.1
- net SWCLK: now reaches IC1.G5 (GPIO[13])
- net SWCLK: now also J1.4 (SWCLK)
- net SWDIO: now reaches IC1.K4 (GPIO[14])
- net SWDIO: now also J1.2 (SWDIO)
- net Peripherals/B_SWITCH: now reaches IC1.K6 (GPIO[55])
- net RF/RF_CNTL_0: now reaches IC1.N3 (RF_CNTL0)
- net RF/RF_CNTL_1: now reaches IC1.P5 (RF_CNTL1)
- net at IC1.R14 (RF_TR_5): now also R5.1
- no-connect marks 11 -> 9
Other:
- sheet Peripherals ports: added B_SWITCH, I2C_SCL, I2C_SDA; removed none
- sheet RF ports: added RF_CNTL_0, RF_CNTL_1; removed VCTL1, VCTL2
- note added: "CON[11] - use SWD"
- moved on the sheet: R1

Commit message: gods greatest decoupler
Parts:
- added C23, C33, C34, C35, C36, C5: 0.1u, Capacitor_SMD:C_0201_0603Metric, symbol Device:C
- added C9: 470p, Capacitor_SMD:C_0201_0603Metric, symbol Device:C
- added R7, R8, R9: 51k, Resistor_SMD:R_0201_0603Metric, symbol Device:R
Connections:
- net +1V0: now also C5.1, C9.1
- net +1V8: now also C23.1, C33.1, C34.1
- net +3V3: now also C35.1, C36.1; no longer C19.1
- net GND: now also C23.2, C33.2, C34.2, C35.2, C36.2, C5.2, C9.2, R7.1, R9.1; no longer IC1.P6 (RF_CNTL2)
- net at IC1.F12 (GPIO[46]): now also R8.1, R9.2
- new net: IC1.P6 (RF_CNTL2), R7.2
- new net +5V: C19.1, R8.2
Other:
- note added: "TPS62840 buck"
- moved on the sheet: C17, C18, C19, C20, C25, C26
