File: HW V1/RW612Implant/rf.kicad_sch (KiCad schematic)
At the start: 11 parts, among them IC2 SKY13323-378LF, U3 SR4W035

Commit message: everything except temp and qi?
Connections:
- net VCTL1 renamed RF_CNTL_0
- net VCTL2 renamed RF_CNTL_1
Other:
- note added: "rf cntl caps?"
Changed lines of the file:
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@@
 	(generator_version "9.0")
 	(paper "A4")
+	(text "rf cntl caps?"
+		(exclude_from_sim no)
+		(at 116.332 61.468 0)
+		(effects
+			(font
+				(size 1.27 1.27)
+			)
+		)
+	)
 	(junction
 		(at 99.06 99.06)
@@
 		)
 	)
-	(hierarchical_label "VCTL1"
+	(hierarchical_label "RF_CNTL_0"
 		(shape input)
 		(at 114.3 64.77 0)
@@
 		)
 	)
-	(hierarchical_label "VCTL2"
+	(hierarchical_label "RF_CNTL_1"
 		(shape input)
 		(at 68.58 72.39 180)

Commit message: gods greatest decoupler
Parts:
- removed C5: 5.6pf, Capacitor_SMD:C_0201_0603Metric, symbol Device:C
Connections:
- net at C6.2, L2.1: now also IC2.5 (INPUT)
Changed lines of the file:
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@@
 	(wire
 		(pts
-			(xy 78.74 88.9) (xy 80.01 88.9)
+			(xy 78.74 88.9) (xy 88.9 88.9)
 		)
 		(stroke
@@
 	(wire
 		(pts
-			(xy 87.63 88.9) (xy 88.9 88.9)
-		)
-		(stroke
-			(width 0)
-			(type default)
-		)
-	)
-	(wire
-		(pts
 			(xy 114.3 72.39) (xy 114.3 73.66)
 		)
@@
 					(unit 1)
 				)
-			)
-		)
-	)
-	(symbol
-		(lib_id "Device:C")
-		(at 83.82 88.9 270)
-		(unit 1)
-		(exclude_from_sim no)
-		(in_bom yes)
-		(on_board yes)
-		(dnp no)
-		(fields_autoplaced yes)
-		(property "Reference" "C5"
-			(at 83.82 81.28 90)
-			(effects
-				(font
-					(size 1.27 1.27)
-				)
-			)
-		)
-		(property "Value" "5.6pf"
-			(at 83.82 83.82 90)
-			(effects
-				(font
-					(size 1.27 1.27)
-				)
-			)
-		)
-		(property "Footprint" "Capacitor_SMD:C_0201_0603Metric"
-			(at 80.01 89.8652 0)
-			(effects
-				(font
-					(size 1.27 1.27)
-				)
-				(hide yes)
-			)
-		)
-		(property "Datasheet" "~"
-			(at 83.82 88.9 0)
-			(effects
-				(font
-					(size 1.27 1.27)
-				)
-				(hide yes)
-			)
-		)
-		(property "Description" "Unpolarized capacitor"
-			(at 83.82 88.9 0)
-			(effects
-				(font
-					(size 1.27 1.27)
-				)
-				(hide yes)
-			)
-		)
-		(pin "1"
-		)
-		(pin "2"
-		)
-		(instances
-			(project "RW612Implant"
-				(path "/a22e6eb7-bd70-4e22-bc03-a0cb284c787e/890467fb-de37-4e48-a756-301e5e4c2a61"
-					(reference "C5")
-					(unit 1)
-				)
