File: NRF54LM20A/NRF54LM20A.kicad_sch (KiCad schematic)
At the start: 30 parts, among them J1 Conn_ARM_SWD_TagConnect_TC203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, U1 S25HS512TFANHI010, U2 nRF54LM20A-QGAA, Y1 CX2016DB32000D0WZRC1

Commit message: straight up routin it
Parts:
- removed C19: 6TPS150MUD, Capacitor_Tantalum_SMD:CP_EIA-3528-21_Kemet-B, symbol Device:C_Polarized
- added C42, C43: TBD, Capacitor_SMD:C_0201_0603Metric, symbol Device:C
- added TP1, TP2, TP3, TP4: RCU-0C, digikey-footprints:PROBE_PAD_0603, symbol dk_Test-Points:RCU-0C
Connections:
- net GND: now also C42.1, C43.1
- net NFC1: now also C43.2, TP3.1
- net NFC2: now also C42.2, TP4.1
- net Peripherals/IMU_SDO: now reaches U2.25 (P0.03)
- net Peripherals/IMU_CS: now reaches U2.13 (P1.03)
- net Peripherals/IMU_INT0: now reaches U2.14 (P1.04)
- net Peripherals/5V_SENSE: now reaches U2.15 (P1.05)
- net Peripherals/5V_SENSE: now also U2.16 (P1.06)
- net Peripherals/IMU_SCK: now reaches U2.22 (P1.07)
- net Peripherals/IMU_INT1: now reaches U2.23 (P1.08)
- net Peripherals/IMU_SDI: now reaches U2.24 (P1.09)
- new net Power/QI_A: TP1.1
- new net Power/QI_B: TP2.1
Other:
- added sheet Power (power.kicad_sch)
- sheet Peripherals ports: added 5V_SENSE, IMU_CS, IMU_INT0, IMU_INT1, IMU_SCK, IMU_SDI, IMU_SDO; removed I2C_SCL, I2C_SDA
- note removed: "TPS62840 buck"
- moved on the sheet: C13, C14
