File: NRF54LM20A/peripherals.kicad_sch (KiCad schematic)
At the start: 5 parts, among them IC3 NMH1000T1, U4 IM67D128BV01, U5 TXS0102DQE

Commit message: straight up routin it
Parts:
- added C40: 0.1u, Capacitor_SMD:C_0201_0603Metric, symbol Device:C
- added R5: 5.1k, Resistor_SMD:R_0201_0603Metric, symbol Device:R
- added R6: 10k, Resistor_SMD:R_0201_0603Metric, symbol Device:R
- added U6: LSM6DSV16B, Package_LGA:LGA-14_3x2.5mm_P0.5mm_LayoutBorder3x4y, symbol New_Library:LSM6DSV16B
Connections:
- net +1V8: now also U6.2 (TDMout), U6.3 (BCLK), U6.5 (VDD_IO), U6.6 (RES), U6.8 (VDD), U6.9 (RES)
- net +5V: now also R6.1
- net GND: now also C40.2, R5.2, U6.7 (GND)
- new net 5V_SENSE: C40.1, R5.1, R6.2
- new net IMU_CS: U6.12 (CS)
- new net IMU_INT0: U6.10 (INT2)
- new net IMU_INT1: U6.4 (INT1)
- new net IMU_SCK: U6.13 (SCL)
- new net IMU_SDI: U6.14 (SDA)
- new net IMU_SDO: U6.1 (SDO/SA0)
- no-connect marks 2 -> 3
Other:
- note removed: "LSM6DSV16B IMU/TEMP"
- note removed: "STTS22H temperature sensor - 3.3v"
